Commit message: add controllers

File: sorter_description/urdf/sorter.xacro (robot description, xacro)
@@ -2,5 +2,5 @@
 <robot name="sorter"
 	xmlns:xacro="http://www.ros.org/wiki/xacro">
-	<!-- Matherials -->
+	<!-- Materials -->
 	<xacro:include filename="$(find sorter_description)/urdf/sorter_materials.xacro" />
 	<!-- abot_base -->
@@ -52,4 +52,6 @@
 		<child link="sorter_base" />
 	</joint>
+	<!-- gazebo plugins -->
+	<xacro:include filename="$(find sorter_description)/urdf/sorter.gazebo" />
 	<!-- Motors -->
 	<xacro:include filename="$(find sorter_description)/urdf/sorter_left_motor.xacro" />
@@ -71,36 +73,3 @@
 	<!-- Sensors -->
 	<xacro:include filename="$(find sorter_description)/urdf/sorter_camera.xacro" />
-	<!-- camera -->
-	<gazebo reference="sorter_camera">
-		<sensor type="camera" name="camera1">
-			<visualize>true</visualize>
-			<update_rate>10.0</update_rate>
-			<camera name="head">
-				<horizontal_fov>1.4</horizontal_fov>
-				<image>
-					<width>600</width>
-					<height>400</height>
-					<format>R8G8B8</format>
-				</image>
-				<clip>
-					<near>0.01</near>
-					<far>0.5</far>
-				</clip>
-			</camera>
-			<plugin name="camera_controller" filename="libgazebo_ros_camera.so">
-				<alwaysOn>true</alwaysOn>
-				<updateRate>0.0</updateRate>
-				<cameraName>sorter/camera1</cameraName>
-				<imageTopicName>image_raw</imageTopicName>
-				<cameraInfoTopicName>camera_info</cameraInfoTopicName>
-				<frameName>sorter_camera</frameName>
-				<hackBaseline>0.07</hackBaseline>
-				<distortionK1>0.0</distortionK1>
-				<distortionK2>0.0</distortionK2>
-				<distortionK3>0.0</distortionK3>
-				<distortionT1>0.0</distortionT1>
-				<distortionT2>0.0</distortionT2>
-			</plugin>
-		</sensor>
-	</gazebo>
 </robot>

File: sorter_description/urdf/sorter_camera.xacro (robot description, xacro)
@@ -29,5 +29,5 @@
   	</gazebo>
   	<joint name="camera2camera_rotate" type="fixed">
-		<origin xyz="0 0.06 0.185" rpy="1.57 -1.57 0"/>
+		<origin xyz="0 0.06 0.185" rpy="-1.57 -1.57 0"/>
 		<parent link="sorter_base"/>
 		<child link="sorter_camera"/>

File: sorter_description/urdf/sorter_left_wheel.xacro (robot description, xacro)
@@ -47,3 +47,13 @@
 		xyz="0 0 1" />
 	</joint>
+	<transmission name="left_wheel_trans">
+	<type>transmission_interface/SimpleTransmission</type>
+	<joint name="left_wheel2motor">
+		<hardwareInterface>hardware_interface/EffortJointInterface</hardwareInterface>
+	</joint>
+	<actuator name="left_wheel_Motor">
+		<hardwareInterface>EffortJointInterface</hardwareInterface>
+		<mechanicalReduction>10</mechanicalReduction>
+	</actuator>
+	</transmission>
 </robot>

File: sorter_description/urdf/sorter_right_wheel.xacro (robot description, xacro)
@@ -47,3 +47,13 @@
 		xyz="1 0 0" />
 	</joint>
+	<transmission name="right_wheel_trans">
+	<type>transmission_interface/SimpleTransmission</type>
+	<joint name="right_wheel2motor">
+		<hardwareInterface>hardware_interface/EffortJointInterface</hardwareInterface>
+	</joint>
+	<actuator name="right_wheel_Motor">
+		<hardwareInterface>EffortJointInterface</hardwareInterface>
+		<mechanicalReduction>10</mechanicalReduction>
+	</actuator>
+	</transmission>
 </robot>
