Commit message: small details

File: sorter_description/urdf/sorter_left_motor.xacro (robot description, xacro)
@@ -11,10 +11,10 @@
 			value="0.10528" />
 			<inertia
-			ixx="0.00010048"
-			ixy="1.3044E-35"
-			ixz="2.6532E-19"
-			iyy="0.00010048"
-			iyz="-3.3687E-21"
-			izz="2.4448E-05" />
+			ixx="0.010048"
+			ixy="1.3044E-33"
+			ixz="2.6532E-17"
+			iyy="0.010048"
+			iyz="-3.3687E-19"
+			izz="2.4448E-03" />
     		</inertial>
 		<visual>

File: sorter_description/urdf/sorter_left_wheel.xacro (robot description, xacro)
@@ -11,10 +11,10 @@
 			value="0.20866" />
 			<inertia
-			ixx="0.0001288"
-			ixy="-9.1557E-13"
-			ixz="1.598E-07"
-			iyy="0.00012883"
-			iyz="-1.6689E-12"
-			izz="8.5081E-05" />
+			ixx="0.01288"
+			ixy="-9.1557E-12"
+			ixz="1.598E-05"
+			iyy="0.012883"
+			iyz="-1.6689E-10"
+			izz="8.5081E-03" />
     		</inertial>
 		<visual>

File: sorter_description/urdf/sorter_right_motor.xacro (robot description, xacro)
@@ -11,10 +11,10 @@
 			value="0.10528" />
 			<inertia
-			ixx="0.00010048"
-			ixy="5.421E-21"
-			ixz="5.9485E-21"
-			iyy="0.00010048"
-			iyz="1.7257E-20"
-			izz="2.4448E-05" />
+			ixx="0.010048"
+			ixy="5.421E-19"
+			ixz="5.9485E-19"
+			iyy="0.010048"
+			iyz="1.7257E-18"
+			izz="2.4448E-03" />
     		</inertial>
 		<visual>

File: sorter_description/urdf/sorter_right_wheel.xacro (robot description, xacro)
@@ -11,10 +11,10 @@
 			value="0.208661050963923" />
 			<inertia
-			ixx="8.50807943773624E-05"
-			ixy="-1.4769453948552E-07"
-			ixz="-6.10195288192908E-08"
-			iyy="0.000128800407810981"
-			iyz="-1.02105267664418E-08"
-			izz="0.000128820903495708" />
+			ixx="8.50807943773624E-03"
+			ixy="-1.4769453948552E-05"
+			ixz="-6.10195288192908E-06"
+			iyy="0.0128800407810981"
+			iyz="-1.02105267664418E-06"
+			izz="0.0128820903495708" />
     		</inertial>
 		<visual>

File: sorter_description/urdf/sorter_scoop.xacro (robot description, xacro)
@@ -11,10 +11,10 @@
 			value="0.15664" />
 			<inertia
-			ixx="0.0030098"
-			ixy="3.2581E-09"
-			ixz="-3.5132E-05"
-			iyy="0.0015134"
-			iyz="5.1464E-08"
-			izz="0.0016037" />
+			ixx="0.30098"
+			ixy="3.2581E-07"
+			ixz="-3.5132E-03"
+			iyy="0.15134"
+			iyz="5.1464E-06"
+			izz="0.16037" />
     		</inertial>
 		<visual>
@@ -52,13 +52,3 @@
 		velocity="0" />
 	</joint>
-	<transmission name="scoop_trans">
-	<type>transmission_interface/SimpleTransmission</type>
-	<joint name="scoop2base">
-		<hardwareInterface>hardware_interface/EffortJointInterface</hardwareInterface>
-	</joint>
-	<actuator name="scoop_Motor">
-		<hardwareInterface>EffortJointInterface</hardwareInterface>
-		<mechanicalReduction>10</mechanicalReduction>
-	</actuator>
-	</transmission>
 </robot>
